Commit message: URDF Viewer Component Updates

File: src/2dofhover/urdf/2dofhover.urdf (robot description, URDF)
Before this commit: robot URDF_V2, 3 links, 2 joints
Links:
- link base_link: geometry collision mesh filename=../meshes/base_link.STL; visual mesh filename=../meshes/base_link.STL
- link link1: geometry collision mesh filename=../meshes/link1.STL; visual mesh filename=../meshes/link1.STL
- link link2: geometry collision mesh filename=../meshes/link2.STL; visual mesh filename=../meshes/link2.STL
